File: Hardware/Microphone-piezo/piezo.kicad_pcb (KiCad board)
At the start: 2 copper layers, 51.5 x 32 mm, 20 parts, among them J1 RJ14, J2 Conn_01x01_Female, J3 Conn_01x01_Female, J4 Conn_01x01_Female, J5 Conn_01x01_Female, U1 NE5534, X1 Piezo

Commit message: Add files via upload
updated files
Parts:
- J2: value Conn_01x01_Female -> conn to ground
Connections:
- J1 pad 3: (no net) -> Net-(J1-Pad3)
- R1 pad 1: Net-(R1-Pad1) -> Net-(D1-Pad2)
- U1 pad 1: (no net) -> Net-(U1-Pad1)
- U1 pad 5: (no net) -> Net-(U1-Pad5)
- U1 pad 8: (no net) -> Net-(U1-Pad8)
- X1 pad 1: Net-(R1-Pad1) -> Net-(D1-Pad2)
Routing:
- net Net-(D1-Pad2): track 6.50 -> 18.5 mm, vias 0 -> 2
- net Net-(R1-Pad1): track 6.50 -> 0.00 mm

Commit message: updated files
Parts:
- added C5: 0.1uF, Capacitor_SMD:CP_Elec_5x5.9, F.Cu at (129.3, 144.0)
- C2: value C -> 47uF
- U1: value NE5534 -> LME49724; footprint Package_SO:SOIC-8_3.9x4.9mm_P1.27mm -> tastatur:PSOIC-8
- moved R4 8.31 mm to (119.6, 136.0)
- moved U1 2.11 mm to (124.5, 133.5)
Connections:
- U1 pad 1: Net-(U1-Pad1) -> Net-(R4-Pad2)
- U1 pad 2: Net-(R4-Pad2) -> Net-(C5-Pad1)
- U1 pad 3: Net-(D1-Pad2) -> VCC
- U1 pad 4: GND -> Net-(R5-Pad1)
- U1 pad 6: Net-(R5-Pad1) -> GND
- U1 pad 8: Net-(U1-Pad8) -> Net-(D1-Pad2)
Routing:
- net GND: track 123.5 -> 0.00 mm, vias 0 -> 3
- net VCC: track 46.6 -> 63.7 mm, vias 0 -> 2
- net Net-(C5-Pad1): track 0.00 -> 15.6 mm
- net Net-(D1-Pad2): track 18.5 -> 29.5 mm, vias 2 -> 0
- net Net-(R4-Pad2): track 12.8 -> 4.98 mm
- net Net-(C4-Pad1): track 29.2 -> 21.4 mm
- net Net-(C1-Pad1): track 30.7 -> 38.3 mm
- net Net-(C3-Pad2): track 8.14 -> 15.5 mm
- net Net-(R5-Pad1): track 8.85 -> 5.75 mm

Commit message: Hopefully the final update
Parts:
- added C6: 10uF, Capacitor_SMD:CP_Elec_5x5.9, F.Cu at (124.7, 122.0)
- added R8: 10K, Resistor_SMD:R_0603_1608Metric_Pad0.98x0.95mm_HandSolder, F.Cu at (126.6, 137.0)
- added R9: 470, Resistor_SMD:R_0603_1608Metric_Pad0.98x0.95mm_HandSolder, F.Cu at (122.6, 128.0)
- U1: footprint tastatur:PSOIC-8 -> piezo:DDA0008B
- moved C2 5.71 mm to (112.8, 143.5), turned to 0 degrees
- moved C3 3.71 mm to (114.3, 123.5), turned to 0 degrees
- moved R4 2.29 mm to (118.5, 134.0)
- moved U1 1.58 mm to (125.0, 132.0)
- moved C5 1.10 mm to (128.2, 144.0)
- moved D1 1.00 mm to (114.5, 136.2)
- moved D2 1.00 mm to (114.5, 130.8)
- moved R1 1.00 mm to (110.5, 133.6)
- moved R2 1.00 mm to (110.5, 137.5)
- moved R3 1.00 mm to (110.5, 129.1)
Connections:
- U1 pad 1: Net-(R4-Pad2) -> Net-(D1-Pad2)
- U1 pad 8: Net-(D1-Pad2) -> Net-(R4-Pad2)
Routing:
- net GND: track 0.00 -> 143.4 mm, vias 3 -> 10
- net Net-(C6-Pad1): track 0.00 -> 20.0 mm
- net Net-(R5-Pad1): track 5.75 -> 15.1 mm, vias 0 -> 2
- net Net-(C1-Pad1): track 38.3 -> 47.0 mm
- net Net-(D1-Pad2): track 29.5 -> 38.2 mm, vias 0 -> 1
- net Net-(C6-Pad2): track 0.00 -> 6.41 mm
- net Net-(C3-Pad2): track 15.5 -> 11.0 mm
- net Net-(R9-Pad2): track 0.00 -> 3.39 mm
- net Net-(R4-Pad2): track 4.98 -> 8.02 mm
- net Net-(C4-Pad1): track 21.4 -> 23.5 mm
- net VCC: track 63.7 -> 64.8 mm, vias 2 -> 1

Commit message: Final update, all should be OK now!
Connections:
- R6 pad 2: Net-(R5-Pad1) -> Net-(R6-Pad2)
- R8 pad 1: Net-(R5-Pad1) -> Net-(R6-Pad2)
- R9 pad 2: Net-(R9-Pad2) -> Net-(R5-Pad1)
- U1 pad 4: Net-(R5-Pad1) -> Net-(R6-Pad2)
- U1 pad 5: Net-(R9-Pad2) -> Net-(R5-Pad1)
Routing:
- net Net-(R6-Pad2): track 0.00 -> 32.0 mm
- net VCC: track 64.8 -> 41.9 mm, vias 1 -> 2
- net Net-(D1-Pad2): track 38.2 -> 48.1 mm, vias 1 -> 0
- net Net-(R9-Pad2): track 3.39 -> 0.00 mm
- net GND: track 143.4 -> 143.6 mm, vias 10 -> 7
